File: xserve-g5.sch (KiCad schematic (older format))
At the start: 4 parts, among them J1 SATA_Backplane_PWR, J2 FAN_LEFT, J3 FAN_RIGHT, J4 PWR

Commit message: update
Parts:
- added J10: FAN5_PWM, Connector_PinSocket_2.54mm:PinSocket_1x04_P2.54mm_Horizontal, symbol Connector_Generic:Conn_01x04
- added J11: FAN6_PWM, Connector_PinSocket_2.54mm:PinSocket_1x04_P2.54mm_Horizontal, symbol Connector_Generic:Conn_01x04
- added J12: FAN7_PWM, Connector_PinSocket_2.54mm:PinSocket_1x04_P2.54mm_Horizontal, symbol Connector_Generic:Conn_01x04
- added J5: PWR_R, Connector_TE-Connectivity:TE_MATE-N-LOK_350211-1_1x04_P5.08mm_Vertical, symbol Connector_Generic:Conn_01x04
- added J6: FAN1_PWM, Connector_PinSocket_2.54mm:PinSocket_1x04_P2.54mm_Horizontal, symbol Connector_Generic:Conn_01x04
- added J7: FAN2_PWM, Connector_PinSocket_2.54mm:PinSocket_1x04_P2.54mm_Horizontal, symbol Connector_Generic:Conn_01x04
- added J8: FAN3_PWM, Connector_PinSocket_2.54mm:PinSocket_1x04_P2.54mm_Horizontal, symbol Connector_Generic:Conn_01x04
- added J9: FAN4_PWM, Connector_PinSocket_2.54mm:PinSocket_1x04_P2.54mm_Horizontal, symbol Connector_Generic:Conn_01x04
- added JP1: PWM1_2, Connector_PinHeader_2.54mm:PinHeader_1x02_P2.54mm_Vertical, symbol Device:Jumper
- added JP2: PWM1_3, Connector_PinHeader_2.54mm:PinHeader_1x02_P2.54mm_Vertical, symbol Device:Jumper
- added JP3: PWM1_4, Connector_PinHeader_2.54mm:PinHeader_1x02_P2.54mm_Vertical, symbol Device:Jumper
- added JP4: PWM5_6, Connector_PinHeader_2.54mm:PinHeader_1x02_P2.54mm_Vertical, symbol Device:Jumper
- added JP5: PWM5_7, Connector_PinHeader_2.54mm:PinHeader_1x02_P2.54mm_Vertical, symbol Device:Jumper
- J4: value PWR -> PWR_L
Connections:
- net labels added: PWM1, PWM2, PWM3, PWM4, PWM5, PWM6, PWM7, TACH1, TACH2, TACH3, TACH4, TACH5, TACH6, TACH7
- net labels removed: +3.3V
- wire segments 14 -> 33
- no-connect marks 2 -> 12
Other:
- note added: "3.3V ??"
- note added: "??"
- moved on the sheet: J1, J2, J3, J4
